Commit message: rework ur5 urdf and adds collision shells for each link

File: arm/configuration/manipulators/ur5/manipulator.urdf (robot description, URDF)
Before this commit: robot ur5_rg2, 12 links, 11 joints
Links:
- link base_link: geometry visual mesh filename=package://robot_simulator/models/ur5_rg2/meshes/visual/ur5/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
- link forearm_link: geometry collision cylinder length=0.425 radius=0.06; visual mesh filename=package://robot_simulator/models/ur5_rg2/meshes/visual/ur5/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
- link rg2_hand: mass 0.29881464108881906 -> None; geometry collision cylinder length=0.14 radius=0.035; visual mesh filename=package://robot_simulator/models/ur5_rg2/meshes/visual/rg2/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
- link rg2_leftfinger: mass 0.24059267945559043 -> None; geometry collision cylinder length=0.1 radius=0.015; visual mesh filename=package://robot_simulator/models/ur5_rg2/meshes/visual/rg2/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
- link rg2_rightfinger: mass 0.24059267945559043 -> None; geometry collision cylinder length=0.1 radius=0.015; visual mesh filename=package://robot_simulator/models/ur5_rg2/meshes/visual/rg2/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
- link shoulder_link: geometry collision cylinder length=0.12 radius=0.08; visual mesh filename=package://robot_simulator/models/ur5_rg2/meshes/visual/ur5/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
- link upper_arm_link: geometry collision cylinder length=0.5 radius=0.08; visual mesh filename=package://robot_simulator/models/ur5_rg2/meshes/visual/ur5/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
- link wrist_1_link: mass 0.8652783044597422 -> None; geometry collision cylinder length=0.1 radius=0.05; visual mesh filename=package://robot_simulator/models/ur5_rg2/meshes/visual/ur5/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
- link wrist_2_link: mass 0.8652786866955592 -> None; geometry collision cylinder length=0.1 radius=0.05; visual mesh filename=package://robot_simulator/models/ur5_rg2/meshes/visual/ur5/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
- link wrist_3_link: mass 0.23285976783205536 -> None; geometry collision cylinder length=0.05 radius=0.05; visual mesh filename=package://robot_simulator/models/ur5_rg2/meshes/visual/ur5/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
Joints:
- joint elbow_joint: origin xyz=0 -0.1197 0.425 rpy=0 0 0 -> xyz=0 -0.1197 0.425
- joint rg2_finger_joint1: limit lower=0.0 upper=1.18 effort=1000.6 velocity=1.57 -> lower=0.0 upper=1.18 effort=1000 velocity=1.57; origin xyz=0.105 0.017 0 rpy=0 0 0 -> xyz=0.105 0.017 0
- joint rg2_finger_joint2: limit lower=0.0 upper=1.18 effort=1000.6 velocity=1.57 -> lower=0.0 upper=1.18 effort=1000 velocity=1.57; origin xyz=0.105 -0.017 0 rpy=0 0 0 -> xyz=0.105 -0.017 0
- joint shoulder_lift_joint: origin xyz=0 0.13585 0 rpy=0 0 0 -> xyz=0 0.13585 0
- joint shoulder_pan_joint: origin xyz=0 0 0.089159 rpy=0 0 0 -> xyz=0 0 0.089159
- joint wrist_1_joint: origin xyz=0 0 0.39225 rpy=0 0 0 -> xyz=0 0 0.39225
- joint wrist_2_joint: origin xyz=0 0.093 0 rpy=0 0 0 -> xyz=0 0.093 0
- joint wrist_3_joint: origin xyz=0 0 0.09465 rpy=0 0 0 -> xyz=0 0 0.09465

Commit message: adds vehicle move action in pick tree

File: arm/configuration/manipulators/ur5/manipulator.urdf (robot description, URDF)
Before this commit: robot ur5_rg2, 12 links, 11 joints
Links:
- link forearm_link: geometry collision cylinder length=0.445 radius=0.07; visual mesh filename=package://robot_simulator/models/ur5_rg2/meshes/visual/ur5/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
- link rg2_hand: geometry collision cylinder length=0.14 radius=0.045; visual mesh filename=package://robot_simulator/models/ur5_rg2/meshes/visual/rg2/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
- link rg2_leftfinger: geometry collision cylinder length=0.1 radius=0.025; visual mesh filename=package://robot_simulator/models/ur5_rg2/meshes/visual/rg2/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
- link rg2_rightfinger: geometry collision cylinder length=0.1 radius=0.025; visual mesh filename=package://robot_simulator/models/ur5_rg2/meshes/visual/rg2/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
- link shoulder_link: geometry collision cylinder length=0.14 radius=0.08; visual mesh filename=package://robot_simulator/models/ur5_rg2/meshes/visual/ur5/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
- link upper_arm_link: geometry collision cylinder length=0.54 radius=0.09; visual mesh filename=package://robot_simulator/models/ur5_rg2/meshes/visual/ur5/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
- link wrist_1_link: geometry collision cylinder length=0.14 radius=0.06; visual mesh filename=package://robot_simulator/models/ur5_rg2/meshes/visual/ur5/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
- link wrist_2_link: geometry collision cylinder length=0.12 radius=0.065; visual mesh filename=package://robot_simulator/models/ur5_rg2/meshes/visual/ur5/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
