Commit message: removes plog, updates kinematics handler to use KDL::Tree

File: arm/arm_bringup/config/manipulators/dxl/manipulator.urdf (robot description, URDF)
Before this commit: robot ur5_rg2, 12 links, 11 joints
Links:
- removed link base_link
- removed link dummy_root
- removed link rg2_hand
- removed link rg2_leftfinger
- removed link rg2_rightfinger
- removed link tool0
- removed link upper_arm_link
- removed link wrist_1_link
- removed link wrist_2_link
- removed link wrist_3_link
- added link gripper_link
- added link left_finger_link; visual mesh filename=package://abv_description/meshes/widow-xl/finger.dae
- added link right_finger_link; visual mesh filename=package://abv_description/meshes/widow-xl/finger.dae
- added link shoulder_mount; visual mesh filename=package://abv_description/meshes/widow-xl/shoulder_mount.dae
- added link widow_xl_base
- added link wrist_link; visual mesh filename=package://abv_description/meshes/widow-xl/wrist.dae
- added link wrist_rotate_link; visual mesh filename=package://abv_description/meshes/widow-xl/wrist_rotate.dae
- link forearm_link: mass 4.210389694173812 -> None; geometry visual mesh filename=package://abv_description/meshes/widow-xl/forearm.dae
- link shoulder_link: mass 2.6078628081050645 -> None; geometry visual mesh filename=package://abv_description/meshes/widow-xl/shoulder.dae
Joints:
- removed joint dummy_root_to_base
- removed joint elbow_joint
- removed joint end_effector_frame_fixed_joint
- removed joint rg2_finger_joint1
- removed joint rg2_finger_joint2
- removed joint shoulder_lift_joint
- removed joint shoulder_pan_joint
- removed joint ur5_hand_joint
- removed joint wrist_1_joint
- removed joint wrist_2_joint
- removed joint wrist_3_joint
- added joint forearm_joint: type revolute, parent shoulder_link, child forearm_link, origin xyz=0.0 -0.0525 0.145 rpy=0 0 0, axis 1 0 0, limit lower=-1.57 upper=1.57 effort=0 velocity=1.0
- added joint gripper_joint: type fixed, parent wrist_rotate_link, child gripper_link, origin xyz=0.0575 0 0 rpy=0 0 0
- added joint left_finger_joint: type prismatic, parent gripper_link, child left_finger_link, origin xyz=0 0.035 0 rpy=0 0 0, axis 0 -1 0, limit lower=0.0 upper=0.0325 effort=10 velocity=1.0
- added joint mount_joint: type fixed, parent widow_xl_base, child shoulder_mount, origin xyz=0 0 0 rpy=0 0 0
- added joint right_finger_joint: type prismatic, parent gripper_link, child right_finger_link, origin xyz=0 -0.035 0 rpy=0 0 0, axis 0 1 0, limit lower=0.0 upper=0.0325 effort=10 velocity=1.0
- added joint shoulder_joint: type revolute, parent shoulder_mount, child shoulder_link, origin xyz=0.0 0.0 0.0 rpy=0 0 0, axis 1 0 0, limit lower=-1.57 upper=1.57 effort=0 velocity=1.0
- added joint wrist_joint: type revolute, parent forearm_link, child wrist_link, origin xyz=0 -0.15 0 rpy=0 0 0, axis 1 0 0, limit lower=-1.57 upper=1.57 effort=0 velocity=1.0
- added joint wrist_rotate_joint: type revolute, parent wrist_link, child wrist_rotate_link, origin xyz=0 -0.075 0 rpy=0 0 -1.57, axis 1 0 0, limit lower=-1.57 upper=1.57 effort=0 velocity=1.0
