Commit message: refactor config structure, extracts gripper from main robot joints for FK/IK and waypoint execution

File: arm/arm_bringup/config/manipulators/ur5/manipulator.urdf (robot description, URDF)
Before this commit: robot ur5_rg2, 12 links, 11 joints
Links:
- removed link base_link
- added link ur5_base_link, mass 4.210389694173812; visual mesh filename=package://robot_simulator/models/ur5_rg2/meshes/visual/ur5/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
Joints:
- joint dummy_root_to_base: child base_link -> ur5_base_link
- joint shoulder_pan_joint: parent base_link -> ur5_base_link
